File: KiCad/PCB/PCB.kicad_sch (KiCad schematic)
At the start: 44 parts

Commit message: PCB Template Design
Parts:
- MX1, MX2, MX3, MX4, MX5, MX6, MX7, MX8, MX9: renamed from MX?; footprint (none) -> MX_Only:MXOnly-1U-NoLED
- R1, R2, R3, R4, R5: renamed from R?; footprint (none) -> Resistor_THT:R_Axial_DIN0207_L6.3mm_D2.5mm_P10.16mm_Horizontal
- R6, R7, R8: renamed from R?; footprint TRIM_PTA4543-2015DPB103 -> Slide Potentiometer:TRIM_PTA4543-2015DPB103
- SW1: renamed from SW?; footprint (none) -> random-keyboard-parts:PushButton_6x6mm_TH_Pretty
- U1: renamed from U?; footprint (none) -> Seeeduino XIAO KICAD:Seeeduino XIAO-MOUDLE14P-2.54-21X17.8MM
- gave numbers to parts that had none: 25
Connections:
- net A0: now also U1.10 (PA5_A9_D9_MISO); no longer U1.1 (PA02_A0_D0)
- net A1: now also U1.9 (PA7_A8_D8_SCK); no longer U1.2 (PA4_A1_D1)
- net A2: now also U1.8 (PB09_A7_D7_RX); no longer U1.3 (PA10_A2_D2)
- net C0: now also U1.1 (PA02_A0_D0); no longer U1.10 (PA5_A9_D9_MISO)
- net C1: now also U1.2 (PA4_A1_D1); no longer U1.9 (PA7_A8_D8_SCK)
- net C2: now also U1.3 (PA10_A2_D2); no longer U1.8 (PB09_A7_D7_RX)
